File: hardware/controller/controller2.sch (EAGLE design)
At the start: 15 parts

Commit message: auto ranging for rotary encoder, a few changes to the chassis, add rangefinder test
Changed lines of the file:
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@@
 <pinref part="P2" gate="A" pin="3"/>
 <wire x1="134.62" y1="-12.7" x2="104.14" y2="-12.7" width="0.1524" layer="91"/>
+<junction x="104.14" y="27.94"/>
 </segment>
 <segment>
