File: hardware/controller/30x70-motor-controller-0.4.brd (EAGLE design)
At the start: 61.1 x 24.9 mm, 19 parts, among them IC1 TS432A-A3G, IC2 TS432A-A3G

Commit message: Lots of controller designs
Parts:
- removed D1: (no value), diode:D-2.5
- removed IC2: TS432A-A3G, assorted:TO92-LINE
- removed R6: 560K, resistor:0204V
- added C3: 1u, resistor:C025-024X044
- added C4: 0.1u, resistor:C025-024X044
- added D2: (no value), diode:D-2.5
- added R3: 10K, resistor:0204V
- added R5: 560k, resistor:0204/7
- C1: device resistor:C050-024X044 -> resistor:C025-025X050
- R2: value 68K -> 100k; device resistor:0207/15 -> resistor:0204V
- R7: value 56K -> 68k
- moved S1 30.9 mm to (7.62, 20.3), turned to 180 degrees
- moved JP1 25.5 mm to (5.08, 2.54)
- moved CN3 24.4 mm to (34.3, 24.1), turned to 0 degrees
- moved CN2 18.0 mm to (43.2, 21.6), turned to 0 degrees
- moved CN1 17.8 mm to (55.9, 21.6), turned to 0 degrees
- moved R4 14.0 mm to (41.9, 10.2), turned to 90 degrees
- moved R2 12.8 mm to (36.8, 5.08), turned to 90 degrees
- moved C1 12.5 mm to (41.9, 5.08), turned to 270 degrees
- moved R7 11.4 mm to (39.4, 10.2)
- moved R1 10.5 mm to (53.3, 14.0)
- moved U$1 10.2 mm to (24.1, 7.62)
- moved U$2 10.2 mm to (53.3, 7.62)
- moved IC1 7.62 mm to (44.5, 14.0)
- moved C2 5.39 mm to (43.2, 16.5), turned to 0 degrees
- moved JP2 5.08 mm to (25.4, 0.00)
Connections:
- new net N$17: C3.1, CN3.2, D2.C, R3.1, S1.1
- net GND: now also CN3.1, S1.3; no longer C1.2, IC2.2, U$2.1
- net N$10: now also D2.A, R2.1, R5.1; no longer C1.1, IC2.3, R6.1
- net N$13: now also IC1.1, U$2.1; no longer D1.A, R7.1
- net N$5: now also C4.1, R3.2; no longer R2.2, U$2.2
- net N$6: now also C3.2, C4.2, U$2.7, U$2.8; no longer IC1.1
- net N$7: no longer U$2.7, U$2.8
- net N$8: now also R7.1; no longer CN3.2, D1.C, S1.3
- net N$9: now also C1.2, R5.2, U$2.2; no longer CN3.1, IC2.1, R2.1, S1.2
- net V+: now also C1.1, R2.2; no longer R6.2
Routing:
- net GND: track 48.3 -> 0.00 mm, vias 2 -> 0
- net N$5: track 35.6 -> 10.2 mm
- net N$8: track 30.5 -> 7.62 mm, vias 2 -> 0
- net N$6: track 5.08 -> 22.9 mm
- net V+: track 38.1 -> 22.9 mm
- net N$7: track 12.7 -> 0.00 mm
- net N$9: track 7.62 -> 0.00 mm
- net N$10: track 5.08 -> 2.54 mm
- net N$17: track 0.00 -> 2.54 mm
- net N$13: track 2.54 -> 0.00 mm
