File: hardware/controller/60x40-motor-controller-0.3.brd (EAGLE design)
At the start: 61.1 x 24.9 mm, 19 parts, among them IC1 TS432A-A3G, IC2 TS432A-A3G

Commit message: Lots of controller designs
Parts:
- added C3: 0.1u, resistor:C025-024X044
- C1: device resistor:C050-024X044 -> resistor:C025-025X050
- D1: device diode:D-2.5 -> diode:D-5
- R1: value 100K -> 82K
- R2: device resistor:0207/15 -> resistor:0204/7
- R6: device resistor:0204V -> resistor:0207/10
- R7: device resistor:0204/7 -> resistor:0204V
- moved R6 23.7 mm to (41.9, 34.3), turned to 180 degrees
- moved R2 20.7 mm to (45.7, 26.7)
- moved IC2 20.3 mm to (44.5, 29.2)
- moved S1 16.6 mm to (35.6, 26.7), turned to 0 degrees
- moved C1 15.3 mm to (45.7, 31.8), turned to 180 degrees
- moved U$2 11.4 mm to (43.2, 12.7), turned to 180 degrees
- moved JP4 11.4 mm to (5.08, 5.08)
- moved CN1 10.2 mm to (45.7, 3.81)
- moved CN3 10.2 mm to (27.9, 0.00)
- moved JP1 10.2 mm to (20.3, 5.08)
- moved JP2 10.2 mm to (15.2, 5.08)
- moved U$1 10.2 mm to (14.0, 17.8)
- moved CN2 10.2 mm to (35.6, 3.81)
- moved C2 4.02 mm to (43.2, 19.1), turned to 0 degrees
- moved R1 3.59 mm to (48.3, 21.6)
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Connections:
- net N$6: now also C2.1, C3.1
- net N$8: now also C3.2, S1.4; no longer C2.1, S1.3
Routing:
- net N$8: track 30.5 -> 7.62 mm, vias 2 -> 0
- net N$6: track 5.08 -> 12.7 mm
- net N$5: track 35.6 -> 30.5 mm
- net GND: track 48.3 -> 43.2 mm, vias 2 -> 0
- net V+: track 38.1 -> 35.6 mm
- net N$9: track 7.62 -> 5.08 mm
Other:
- board size 61.1 x 24.9 mm -> 50.8 x 35.6 mm
